File: discipline-pcb.kicad_pcb (KiCad board)
At the start: 2 copper layers, 304.9 x 122.8 mm, 180 parts, among them J1 AVR-ISP-6, SW1 KEYSW, SW10 KEYSW, SW11 KEYSW, SW12 KEYSW, SW13 KEYSW, SW14 KEYSW, SW15 KEYSW, SW16 KEYSW, SW17 KEYSW, SW18 KEYSW, SW19 KEYSW, SW2 KEYSW, SW20 KEYSW, SW21 KEYSW, SW22 KEYSW, SW23 KEYSW, SW24 KEYSW, SW25 KEYSW, SW26 KEYSW, SW27 KEYSW, SW28 KEYSW, SW29 KEYSW, SW3 KEYSW, SW30 KEYSW, SW31 KEYSW, SW32 KEYSW, SW33 KEYSW, SW34 KEYSW, SW35 KEYSW, SW36 KEYSW, SW37 KEYSW, SW38 KEYSW, SW39 KEYSW, SW4 KEYSW, SW40 KEYSW, SW41 KEYSW, SW42 KEYSW, SW43 KEYSW, SW44 KEYSW, SW45 KEYSW, SW46 KEYSW, SW47 KEYSW, SW48 KEYSW, SW49 KEYSW, SW5 KEYSW, SW50 KEYSW, SW51 KEYSW, SW52 KEYSW, SW53 KEYSW, SW54 KEYSW, SW55 KEYSW, SW56 KEYSW, SW57 KEYSW, SW58 KEYSW, SW59 KEYSW, SW6 KEYSW, SW60 KEYSW, SW61 KEYSW, SW62 KEYSW, SW63 KEYSW, SW64 KEYSW, SW65 KEYSW, SW66 KEYSW, SW67 KEYSW, SW68 KEYSW, SW69 KEYSW, SW7 KEYSW, SW70 KEYSW, SW71 KEYSW, SW72 KEYSW, SW73 KEYSW, SW74 KEYSW, SW8 KEYSW, SW9 KEYSW, U1 ATmega32A-PU, Y1 Crystal

Commit message: Discipline ISO
Parts:
- added D45A2: , cftkb:D_DO-35_SOD27_P5.08mm_Horizontal, F.Cu at (60.5, 66.2)
- added SW29A1: KEYSW, cftkb:SW_Cherry_MX1A_1.00u_PCB-NOSCREEN, F.Cu at (308.7, 127.8)
- added SW43A1: KEYSW, cftkb:SW_Cherry_MX1A_2.00u_PCBNOSCREEN, F.Cu at (332.7, 125.9)
- added SW45A1: KEYSW, cftkb:SW_Cherry_MX1A_1.25u_PCBNOSCREEN, F.Cu at (68.3, 146.9)
- added SW45A2: KEYSW, cftkb:SW_Cherry_MX1A_1.00u_PCB-NOSCREEN, F.Cu at (89.7, 146.9)
- moved G*** 1.35 mm to (57.1, 71.1)
Routing:
- net Net-(D45A2-Pad2): track 0.00 -> 151.9 mm
- net Net-(D29-Pad2): track 117.7 -> 149.3 mm
- net col13: track 146.9 -> 169.7 mm
- net Net-(D43-Pad2): track 140.6 -> 161.8 mm
- net row3: track 287.2 -> 302.5 mm
- net col1: track 317.2 -> 330.7 mm
- net Net-(D45-Pad2): track 76.5 -> 86.0 mm
- net col0: track 355.0 -> 361.8 mm
- net col12: track 182.7 -> 186.9 mm
- net Net-(D64-Pad2): track 187.5 -> 189.5 mm
- net Net-(D56-Pad2): track 145.3 -> 146.7 mm
- net GND: vias 36 -> 38
