File: discipline-pcb.sch (KiCad schematic (older format))
At the start: 164 parts, among them J1 AVR-ISP-6, SW1 KEYSW, SW10 KEYSW, SW11 KEYSW, SW12 KEYSW, SW13 KEYSW, SW14 KEYSW, SW15 KEYSW, SW16 KEYSW, SW17 KEYSW, SW18 KEYSW, SW19 KEYSW, SW2 KEYSW, SW20 KEYSW, SW21 KEYSW, SW22 KEYSW, SW23 KEYSW, SW24 KEYSW, SW25 KEYSW, SW26 KEYSW, SW27 KEYSW, SW28 KEYSW, SW29 KEYSW, SW3 KEYSW, SW30 KEYSW, SW31 KEYSW, SW32 KEYSW, SW33 KEYSW, SW34 KEYSW, SW35 KEYSW, SW36 KEYSW, SW37 KEYSW, SW38 KEYSW, SW39 KEYSW, SW4 KEYSW, SW40 KEYSW, SW41 KEYSW, SW42 KEYSW, SW43 KEYSW, SW44 KEYSW, SW45 KEYSW, SW46 KEYSW, SW47 KEYSW, SW48 KEYSW, SW49 KEYSW, SW5 KEYSW, SW50 KEYSW, SW51 KEYSW, SW52 KEYSW, SW53 KEYSW, SW54 KEYSW, SW55 KEYSW, SW56 KEYSW, SW57 KEYSW, SW58 KEYSW, SW59 KEYSW, SW6 KEYSW, SW60 KEYSW, SW61 KEYSW, SW62 KEYSW, SW63 KEYSW, SW64 KEYSW, SW65 KEYSW, SW66 KEYSW, SW67 KEYSW, SW68 KEYSW, SW69 KEYSW, SW7 KEYSW, SW70 KEYSW, SW71 KEYSW, SW72 KEYSW, SW73 KEYSW, SW74 KEYSW, SW8 KEYSW, SW9 KEYSW, U1 ATmega32A-PU, Y1 Crystal

Commit message: Discipline ISO
Parts:
- added D45A2: (no value), cftkb:D_DO-35_SOD27_P5.08mm_Horizontal, symbol discipline-pcb-rescue:D-Device
- added SW29A1, SW45A2: KEYSW, cftkb:SW_Cherry_MX1A_1.00u_PCB-NOSCREEN, symbol discipline-pcb-rescue:KEYSW-keyboard_parts
- added SW43A1: KEYSW, cftkb:SW_Cherry_MX1A_2.00u_PCBNOSCREEN, symbol discipline-pcb-rescue:KEYSW-keyboard_parts
- added SW45A1: KEYSW, cftkb:SW_Cherry_MX1A_1.25u_PCBNOSCREEN, symbol discipline-pcb-rescue:KEYSW-keyboard_parts
- BOOT1, RESET1: symbol keyboard_parts:SW_PUSH -> discipline-pcb-rescue:SW_PUSH-keyboard_parts
- C1, C2, C4, C5: symbol Device:C_Small -> discipline-pcb-rescue:C_Small-Device
- C3: symbol Device:CP1_Small -> discipline-pcb-rescue:CP1_Small-Device
- D1, D10, D11, D12, D13, D14, D15, D16, D17, D18, D19, D2, D20, D21, D22, D23, D24, D25, D26, D27, D28, D29, D3, D30, D31, D32, D33, D34, D35, D36, D37, D38, D39, D4, D40, D41, D42, D43, D44, D45, D46, D47, D48, D49, D5, D50, D51, D52, D53, D54, D55, D56, D57, D58, D59, D6, D60, D61, D62, D63, D64, D65, D66, D67, D68, D7, D8, D9: symbol Device:D -> discipline-pcb-rescue:D-Device
- D69, D70: symbol Device:D_Zener_Small -> discipline-pcb-rescue:D_Zener_Small-Device
- F1: symbol Device:Polyfuse_Small -> discipline-pcb-rescue:Polyfuse_Small-Device
- J1: symbol Connector:AVR-ISP-6 -> discipline-pcb-rescue:AVR-ISP-6-Connector
- LED1: symbol Device:LED -> discipline-pcb-rescue:LED-Device
- R1, R2, R3, R4, R5, R6, R7: symbol Device:R_Small -> discipline-pcb-rescue:R_Small-Device
- SW1, SW10, SW11, SW12, SW13, SW14, SW15, SW16, SW17, SW18, SW19, SW2, SW20, SW21, SW22, SW23, SW24, SW25, SW26, SW27, SW28, SW29, SW3, SW30, SW31, SW32, SW33, SW34, SW35, SW36, SW37, SW38, SW39, SW4, SW40, SW41, SW42, SW43, SW44, SW45, SW46, SW47, SW48, SW49, SW5, SW50, SW51, SW52, SW53, SW54, SW55, SW56, SW57, SW58, SW59, SW6, SW60, SW61, SW62, SW63, SW64, SW65, SW66, SW67, SW68, SW69, SW7, SW70, SW71, SW72, SW73, SW74, SW8, SW9: symbol keyboard_parts:KEYSW -> discipline-pcb-rescue:KEYSW-keyboard_parts
- U1: symbol MCU_Microchip_ATmega:ATmega32A-PU -> discipline-pcb-rescue:ATmega32A-PU-MCU_Microchip_ATmega
- USB1: symbol Type-C:USB_C_GCT_USB4085 -> discipline-pcb-rescue:USB_C_GCT_USB4085-Type-C
- Y1: symbol Device:Crystal -> discipline-pcb-rescue:Crystal-Device
Connections:
- wire segments 342 -> 354
